Commit message: Fine Tuned

File: motoman/motoman_motomini_support/urdf/gripper_macro.xacro (robot description, xacro)
@@ -28,4 +28,9 @@
       </geometry>
     </collision>
+        <inertial>
+        <origin xyz="0 0 0" rpy="0 0 0" />
+        <mass value= "0.1"/>
+        <inertia ixx="0.001" ixy="0.001" ixz="0.001" iyy="0.001" iyz="0.001" izz="0.001" />
+    </inertial>
   </link>
   <link name="claw_1a">
@@ -41,4 +46,9 @@
       </geometry>
     </collision>
+        <inertial>
+        <origin xyz="0 0 0" rpy="0 0 0" />
+        <mass value= "0.1"/>
+        <inertia ixx="0.001" ixy="0.001" ixz="0.001" iyy="0.001" iyz="0.001" izz="0.001" />
+    </inertial>
   </link>
   <link name="claw_1b">
@@ -54,4 +64,9 @@
       </geometry>
     </collision>
+        <inertial>
+        <origin xyz="0 0 0" rpy="0 0 0" />
+        <mass value= "0.1"/>
+        <inertia ixx="0.001" ixy="0.001" ixz="0.001" iyy="0.001" iyz="0.001" izz="0.001" />
+    </inertial>
   </link>
   <link name="claw_2a">
@@ -67,4 +82,9 @@
       </geometry>
     </collision>
+        <inertial>
+        <origin xyz="0 0 0" rpy="0 0 0" />
+        <mass value= "0.1"/>
+        <inertia ixx="0.001" ixy="0.001" ixz="0.001" iyy="0.001" iyz="0.001" izz="0.001" />
+    </inertial>
   </link>
   <link name="claw_2b">
@@ -80,4 +100,9 @@
       </geometry>
     </collision>
+        <inertial>
+        <origin xyz="0 0 0" rpy="0 0 0" />
+        <mass value= "0.1"/>
+        <inertia ixx="0.001" ixy="0.001" ixz="0.001" iyy="0.001" iyz="0.001" izz="0.001" />
+    </inertial>
   </link>
   <link name="link_1a">
@@ -93,4 +118,9 @@
       </geometry>
     </collision>
+        <inertial>
+        <origin xyz="0 0 0" rpy="0 0 0" />
+        <mass value= "0.1"/>
+        <inertia ixx="0.001" ixy="0.001" ixz="0.001" iyy="0.001" iyz="0.001" izz="0.001" />
+    </inertial>
   </link>
   <link name="link_1b">
@@ -106,4 +136,9 @@
       </geometry>
     </collision>
+        <inertial>
+        <origin xyz="0 0 0" rpy="0 0 0" />
+        <mass value= "0.1"/>
+        <inertia ixx="0.001" ixy="0.001" ixz="0.001" iyy="0.001" iyz="0.001" izz="0.001" />
+    </inertial>
   </link>
   <link name="link_2a">
@@ -119,4 +154,9 @@
       </geometry>
     </collision>
+        <inertial>
+        <origin xyz="0 0 0" rpy="0 0 0" />
+        <mass value= "0.1"/>
+        <inertia ixx="0.001" ixy="0.001" ixz="0.001" iyy="0.001" iyz="0.001" izz="0.001" />
+    </inertial>
   </link>
     <link name="link_2b">
@@ -132,4 +172,9 @@
       </geometry>
     </collision>
+        <inertial>
+        <origin xyz="0 0 0" rpy="0 0 0" />
+        <mass value= "0.1"/>
+        <inertia ixx="0.001" ixy="0.001" ixz="0.001" iyy="0.001" iyz="0.001" izz="0.001" />
+    </inertial>
   </link>
     <link name="link_2c">
@@ -145,4 +190,9 @@
       </geometry>
     </collision>
+        <inertial>
+        <origin xyz="0 0 0" rpy="0 0 0" />
+        <mass value= "0.1"/>
+        <inertia ixx="0.001" ixy="0.001" ixz="0.001" iyy="0.001" iyz="0.001" izz="0.001" />
+    </inertial>
   </link>
     <link name="link_2d">
@@ -158,5 +208,28 @@
       </geometry>
     </collision>
-  </link>
+        <inertial>
+        <origin xyz="0 0 0" rpy="0 0 0" />
+        <mass value= "0.1"/>
+        <inertia ixx="0.001" ixy="0.001" ixz="0.001" iyy="0.001" iyz="0.001" izz="0.001" />
+    </inertial>
+  </link>
+      <!--link name="servo_motor">
+    <visual>
+      <geometry>
+        <box size="0.054 0.020 0.038"/>
+      </geometry>
+      <material name="white"/>
+    </visual>
+    <collision>
+      <geometry>
+        <box size="0.054 0.020 0.038"/>
+      </geometry>
+    </collision>
+        <inertial>
+        <origin xyz="0 0 0" rpy="0 0 0" />
+        <mass value= "0.1"/>
+        <inertia ixx="0.001" ixy="0.001" ixz="0.001" iyy="0.001" iyz="0.001" izz="0.001" />
+    </inertial>
+  </link-->
 <joint name="gripper_joint" type="fixed">
     <parent link="${parent}"/>
@@ -246,4 +319,9 @@
     <mimic joint="claw_1b_joint" multiplier="1"/>
   </joint>
+<!--joint name="servo_joint" type="fixed">
+    <parent link="gripper_base"/>
+    <child link="servo_motor"/>
+    <origin rpy="0.0 0.0 1.5707" xyz="0.062257 0.0040985 0"/>
+  </joint-->
     </xacro:macro>
 </robot>

File: motoman/motoman_motomini_support/urdf/motomini.urdf (robot description, URDF)
Before this commit: robot motoman_motomini, 12 links, 11 joints
Links:
- removed link kinect2_link
- added link camera_link; collision box size=0.05 0.2 0.05; visual box size=0.05 0.2 0.05
- added link claw_1a; collision mesh filename=package://motoman_motomini_support/meshes/gripper/claw_1.stl; visual mesh filename=package://motoman_motomini_support/meshes/gripper/claw_1.stl
- added link claw_1b; collision mesh filename=package://motoman_motomini_support/meshes/gripper/claw_1.stl; visual mesh filename=package://motoman_motomini_support/meshes/gripper/claw_1.stl
- added link claw_2a; collision mesh filename=package://motoman_motomini_support/meshes/gripper/claw_2.stl; visual mesh filename=package://motoman_motomini_support/meshes/gripper/claw_2.stl
- added link claw_2b; collision mesh filename=package://motoman_motomini_support/meshes/gripper/claw_2.stl; visual mesh filename=package://motoman_motomini_support/meshes/gripper/claw_2.stl
- added link gripper_base; collision mesh filename=package://motoman_motomini_support/meshes/gripper/base.stl; visual mesh filename=package://motoman_motomini_support/meshes/gripper/base.stl
- added link link_1a; collision mesh filename=package://motoman_motomini_support/meshes/gripper/link_1.stl; visual mesh filename=package://motoman_motomini_support/meshes/gripper/link_1.stl
- added link link_1b; collision mesh filename=package://motoman_motomini_support/meshes/gripper/link_1.stl; visual mesh filename=package://motoman_motomini_support/meshes/gripper/link_1.stl
- added link link_2a; collision mesh filename=package://motoman_motomini_support/meshes/gripper/link_2.stl; visual mesh filename=package://motoman_motomini_support/meshes/gripper/link_2.stl
- added link link_2b; collision mesh filename=package://motoman_motomini_support/meshes/gripper/link_2.stl; visual mesh filename=package://motoman_motomini_support/meshes/gripper/link_2.stl
- added link link_2c; collision mesh filename=package://motoman_motomini_support/meshes/gripper/link_2.stl; visual mesh filename=package://motoman_motomini_support/meshes/gripper/link_2.stl
- added link link_2d; collision mesh filename=package://motoman_motomini_support/meshes/gripper/link_2.stl; visual mesh filename=package://motoman_motomini_support/meshes/gripper/link_2.stl
- added link realsense_link, mass 1e-5; collision box size=0.001 0.001 0.001; visual mesh filename=package://ebot_description/meshes/NAVRS.STL
- added link tool_tip
Joints:
- added joint claw_1a_joint: type revolute, parent gripper_base, child claw_1a, origin xyz=0.045 -0.01154 0.017503 rpy=0.0 0.0 -1.3386, axis 0 0 1, limit lower=-3.0 upper=3.0 effort=200 velocity=3, mimic joint=claw_1b_joint multiplier=-1
- added joint claw_1b_joint: type revolute, parent gripper_base, child claw_1b, origin xyz=0.045 0.01154 0.017503 rpy=0.0 0.0 1.3386, axis 0 0 1, limit lower=-3.0 upper=3.0 effort=200 velocity=3
- added joint claw_2a_joint: type revolute, parent claw_1a, child claw_2a, origin xyz=0.03 0 -0.005 rpy=3.142 0 -1.6029994, axis 0 0 1, limit lower=-3.0 upper=3.0 effort=200 velocity=3, mimic joint=claw_1b_joint multiplier=-1
- added joint claw_2b_joint: type revolute, parent claw_1b, child claw_2b, origin xyz=0.03 0 -0.005 rpy=3.142 3.142 -1.6029994, axis 0 0 1, limit lower=-3.0 upper=3.0 effort=200 velocity=3, mimic joint=claw_1b_joint multiplier=-1
- added joint gripper_joint: type fixed, parent tool0, child gripper_base, origin xyz=0 0 0 rpy=0 -1.5707 3.142
- added joint gripper_tip: type fixed, parent tool0, child tool_tip, origin xyz=0.012 0 0.115  rpy=3.14159265359 -1.57079632679 0
- added joint link_1a_joint: type revolute, parent gripper_base, child link_1a, origin xyz=0.045 -0.01154 0.0044 rpy=0.0 0.0 1.8033928, axis 0 0 1, limit lower=-3.0 upper=3.0 effort=200 velocity=3, mimic joint=claw_1b_joint multiplier=-1
- added joint link_1b_joint: type revolute, parent gripper_base, child link_1b, origin xyz=0.045 0.01154 0.0044 rpy=0.0 0.0 -1.8033928, axis 0 0 1, limit lower=-3.0 upper=3.0 effort=200 velocity=3, mimic joint=claw_1b_joint multiplier=1
- added joint link_2a_joint: type revolute, parent gripper_base, child link_2a, origin xyz=0.062257 -0.0040985 0.02 rpy=0.0 0.0 1.8033928, axis 0 0 1, limit lower=-3.0 upper=3.0 effort=200 velocity=3, mimic joint=claw_1b_joint multiplier=-1
- added joint link_2b_joint: type revolute, parent gripper_base, child link_2b, origin xyz=0.062257 0.0040985 0.02 rpy=0.0 0.0 -1.8033928, axis 0 0 1, limit lower=-3.0 upper=3.0 effort=200 velocity=3, mimic joint=claw_1b_joint multiplier=1
- added joint link_2c_joint: type revolute, parent gripper_base, child link_2c, origin xyz=0.062257 -0.0040985 0.005 rpy=0.0 0.0 1.8033928, axis 0 0 1, limit lower=-3.0 upper=3.0 effort=200 velocity=3, mimic joint=claw_1b_joint multiplier=-1
- added joint link_2d_joint: type revolute, parent gripper_base, child link_2d, origin xyz=0.062257 0.0040985 0.005 rpy=0.0 0.0 -1.8033928, axis 0 0 1, limit lower=-3.0 upper=3.0 effort=200 velocity=3, mimic joint=claw_1b_joint multiplier=1
- added joint realsense_joint: type fixed, parent gripper_base, child realsense_link, origin xyz=0.05 0 0.055 rpy=0 0 0
- joint camera_joint: child kinect2_link -> camera_link; origin xyz=0.865 0 0.525 rpy=-2.042 0 1.57079632679 -> xyz=1.17 0 0.48 rpy=0 0.4712 -3.14159265359

File: motoman/motoman_motomini_support/urdf/motomini.xacro (robot description, xacro)
@@ -1,11 +1,21 @@
 <?xml version="1.0" ?>
 <robot name="motoman_motomini" xmlns:xacro="http://ros.org/wiki/xacro">
+  <xacro:include filename="$(find motoman_motomini_support)/urdf/motomini_gazebo.xacro" />
+  <xacro:property name="M_PI" value="3.1415926535897931" />
+  <xacro:include filename="$(find motoman_motomini_support)/urdf/table_macro.xacro" />
   <xacro:include filename="$(find motoman_motomini_support)/urdf/motomini_macro_kinect1.xacro" />
-  <xacro:motoman_motomini prefix=""/>
   <xacro:include filename="$(find motoman_motomini_support)/urdf/gripper_macro.xacro" />
+  <xacro:include filename="$(find motoman_motomini_support)/urdf/realsense_macro.xacro" />
+   <!-- World frame -->
+  <link name="world" />
+  <xacro:motoman_motomini_table prefix="" parent="world">
+  	<origin xyz="0 0 0" rpy="0 0 -${M_PI/2}" />
+  </xacro:motoman_motomini_table>
+  <xacro:motoman_motomini prefix="" parent="table">
+  <origin xyz="0 -0.1015 0.0" rpy="0.0 0.0 ${M_PI/2}" />
+  </xacro:motoman_motomini>
   <xacro:motoman_motomini_gripper prefix="" parent="tool0">
-  	<origin xyz="0 0 0" rpy="0 -1.5707 3.142" />
+  	<origin xyz="0 0 0" rpy="0 -${M_PI/2} ${M_PI}" />
   </xacro:motoman_motomini_gripper>
-  <xacro:include filename="$(find motoman_motomini_support)/urdf/realsense_macro.xacro" />
   <xacro:motoman_motomini_realsense prefix="" parent="gripper_base">
   	<origin xyz="0.05 0 0.055" rpy="0 0 0" />
