Commit message: Fixed height

File: motoman/motoman_motomini_support/urdf/table_macro.xacro (robot description, xacro)
@@ -11,5 +11,5 @@
     <visual>
       <geometry>
-        <box size="0.83 0.830 0.001"/>
+        <mesh filename="package://motoman_motomini_support/urdf/table.dae"/>
       </geometry>
         <material name = "light_grey">
@@ -19,89 +19,5 @@
     <collision>
       <geometry>
-         <box size="0.83 0.830 0.001"/>
-      </geometry>
-    </collision>
-  </link>
-<link name="leg1">
-  <origin xyz="0.0 0.0 0" rpy="0 0 0" />
-  <inertial>
-          <mass value="1" />
-          <origin xyz="0 0 0" />
-          <inertia ixx="1" ixy="0.0" ixz="0.0" iyy="1" iyz="0.0" izz="1" />
-    </inertial>
-    <visual>
-      <geometry>
-        <box size="0.03 0.03 0.7"/>
-      </geometry>
-        <material name = "light_grey">
-         <color rgba="0.7 0.7 0.7 1.0"/>
-        </material>
-    </visual>
-    <collision>
-      <geometry>
-         <box size="0.03 0.03 0.7"/>
-      </geometry>
-    </collision>
-  </link>
-<link name="leg2">
-  <origin xyz="0.0 0.0 0" rpy="0 0 0" />
-  <inertial>
-          <mass value="1" />
-          <origin xyz="0 0 0" />
-          <inertia ixx="1" ixy="0.0" ixz="0.0" iyy="1" iyz="0.0" izz="1" />
-    </inertial>
-    <visual>
-      <geometry>
-        <box size="0.03 0.03 0.7"/>
-      </geometry>
-        <material name = "light_grey">
-         <color rgba="0.7 0.7 0.7 1.0"/>
-        </material>
-    </visual>
-    <collision>
-      <geometry>
-         <box size="0.03 0.03 0.7"/>
-      </geometry>
-    </collision>
-  </link>
-<link name="leg3">
-  <origin xyz="0.0 0.0 0" rpy="0 0 0" />
-  <inertial>
-          <mass value="1" />
-          <origin xyz="0 0 0" />
-          <inertia ixx="1" ixy="0.0" ixz="0.0" iyy="1" iyz="0.0" izz="1" />
-    </inertial>
-    <visual>
-      <geometry>
-        <box size="0.03 0.03 0.7"/>
-      </geometry>
-        <material name = "light_grey">
-         <color rgba="0.7 0.7 0.7 1.0"/>
-        </material>
-    </visual>
-    <collision>
-      <geometry>
-         <box size="0.03 0.03 0.7"/>
-      </geometry>
-    </collision>
-  </link>
-<link name="leg4">
-  <origin xyz="0.0 0.0 0" rpy="0 0 0" />
-  <inertial>
-          <mass value="1" />
-          <origin xyz="0 0 0" />
-          <inertia ixx="1" ixy="0.0" ixz="0.0" iyy="1" iyz="0.0" izz="1" />
-    </inertial>
-    <visual>
-      <geometry>
-        <box size="0.03 0.03 0.7"/>
-      </geometry>
-        <material name = "light_grey">
-         <color rgba="0.7 0.7 0.7 1.0"/>
-        </material>
-    </visual>
-    <collision>
-      <geometry>
-         <box size="0.03 0.03 0.7"/>
+         <mesh filename="package://motoman_motomini_support/urdf/table.dae"/>
       </geometry>
     </collision>
@@ -114,24 +30,4 @@
     <axis xyz = "0 0 1" />-->
 </joint>
-  <joint name="leg1_joint" type="fixed">
-    <parent link="table"/>
-    <child link="leg1"/>
-    <origin rpy="0.0 0.0 0" xyz="0.4 0.4 -0.35"/>
-  </joint>
-  <joint name="leg2_joint" type="fixed">
-    <parent link="table" />
-    <child link = "leg2" />
-    <origin xyz="0.4 -0.4 -0.35" rpy="0 0 0" />
-  </joint>
-  <joint name="leg3_joint" type="fixed">
-    <parent link="table"/>
-    <child link="leg3"/>
-    <origin xyz="-0.4 0.4 -0.35" rpy="0 0 0" />
-  </joint>
-  <joint name="leg4_joint" type="fixed">
-    <parent link="table"/>
-    <child link="leg4"/>
-    <origin xyz="-0.4 -0.4 -0.35" rpy="0 0 0" />
-  </joint>
-    </xacro:macro>
+</xacro:macro>
 </robot>

File: motoman/motoman_motomini_support/urdf_old/gripper_macro.xacro (robot description, xacro)
@@ -324,124 +324,4 @@
     <origin rpy="0.0 0.0 1.5707" xyz="0.062257 0.0040985 0"/>
   </joint-->
-<gazebo reference="gripper_base">
-    <implicitSpringDamper>1</implicitSpringDamper>
-    <kp>1000000.0</kp>
-    <kd>1.0</kd>
-    <mu1>10000.0</mu1>
-    <mu2>10000.0</mu2>
-    <minDepth>0.001</minDepth>
-<material>Gazebo/Black</material>
-    <turnGravityOff>false</turnGravityOff>
-</gazebo>
-<gazebo reference="claw_1a">
-    <implicitSpringDamper>1</implicitSpringDamper>
-    <kp>1000000.0</kp>
-    <kd>1.0</kd>
-    <mu1>10000.0</mu1>
-    <mu2>10000.0</mu2>
-    <minDepth>0.001</minDepth>
-<material>Gazebo/Black</material>
-    <turnGravityOff>false</turnGravityOff>
-</gazebo>
-<gazebo reference="claw_1b">
-    <implicitSpringDamper>1</implicitSpringDamper>
-    <kp>1000000.0</kp>
-    <kd>1.0</kd>
-    <mu1>10000.0</mu1>
-    <mu2>10000.0</mu2>
-    <minDepth>0.001</minDepth>
-<material>Gazebo/Black</material>
-    <turnGravityOff>false</turnGravityOff>
-</gazebo>
-<gazebo reference="claw_2a">
-    <implicitSpringDamper>1</implicitSpringDamper>
-    <kp>1000000.0</kp>
-    <kd>1.0</kd>
-    <mu1>10000.0</mu1>
-    <mu2>10000.0</mu2>
-    <minDepth>0.001</minDepth>
-<material>Gazebo/Black</material>
-    <turnGravityOff>false</turnGravityOff>
-</gazebo>
-<gazebo reference="claw_2b">
-    <implicitSpringDamper>1</implicitSpringDamper>
-    <kp>1000000.0</kp>
-    <kd>1.0</kd>
-    <mu1>10000.0</mu1>
-    <mu2>10000.0</mu2>
-    <minDepth>0.001</minDepth>
-<material>Gazebo/Black</material>
-    <turnGravityOff>false</turnGravityOff>
-</gazebo>
-<gazebo reference="link_1a">
-    <implicitSpringDamper>1</implicitSpringDamper>
-    <kp>1000000.0</kp>
-    <kd>1.0</kd>
-    <mu1>10000.0</mu1>
-    <mu2>10000.0</mu2>
-    <minDepth>0.001</minDepth>
-<material>Gazebo/Black</material>
-    <turnGravityOff>false</turnGravityOff>
-</gazebo>
-<gazebo reference="link_1b">
-    <implicitSpringDamper>1</implicitSpringDamper>
-    <kp>1000000.0</kp>
-    <kd>1.0</kd>
-    <mu1>10000.0</mu1>
-    <mu2>10000.0</mu2>
-    <minDepth>0.001</minDepth>
-<material>Gazebo/Black</material>
-    <turnGravityOff>false</turnGravityOff>
-</gazebo>
-<gazebo reference="link_2a">
-    <implicitSpringDamper>1</implicitSpringDamper>
-    <kp>1000000.0</kp>
-    <kd>1.0</kd>
-    <mu1>10000.0</mu1>
-    <mu2>10000.0</mu2>
-    <minDepth>0.001</minDepth>
-<material>Gazebo/Black</material>
-    <turnGravityOff>false</turnGravityOff>
-</gazebo>
-<gazebo reference="link_2b">
-    <implicitSpringDamper>1</implicitSpringDamper>
-    <kp>1000000.0</kp>
-    <kd>1.0</kd>
-    <mu1>10000.0</mu1>
-    <mu2>10000.0</mu2>
-    <minDepth>0.001</minDepth>
-<material>Gazebo/Black</material>
-    <turnGravityOff>false</turnGravityOff>
-</gazebo>
-<gazebo reference="link_2c">
-    <implicitSpringDamper>1</implicitSpringDamper>
-    <kp>1000000.0</kp>
-    <kd>1.0</kd>
-    <mu1>10000.0</mu1>
-    <mu2>10000.0</mu2>
-    <minDepth>0.001</minDepth>
-<material>Gazebo/Black</material>
-    <turnGravityOff>false</turnGravityOff>
-</gazebo>
-<gazebo reference="link_2d">
-    <implicitSpringDamper>1</implicitSpringDamper>
-    <kp>1000000.0</kp>
-    <kd>1.0</kd>
-    <mu1>100000</mu1>
-    <mu2>100000</mu2>
-    <minDepth>0.001</minDepth>
- <material>Gazebo/Black</material>
-    <turnGravityOff>false</turnGravityOff>
-</gazebo>
-<transmission name="link5_finger1_control">
-    <type>transmission_interface/SimpleTransmission</type>
-    <joint name="claw_1b_joint">
-     <hardwareInterface>hardware_interface/PositionJointInterface</hardwareInterface>
-    </joint>
-    <actuator name="l_finger_motor">
-     <hardwareInterface>hardware_interface/PositionJointInterface</hardwareInterface>
-     <mechanicalReduction>2</mechanicalReduction>
-    </actuator>
-</transmission>
     </xacro:macro>
 </robot>

File: motoman/motoman_motomini_support/urdf_old/motoman_motomini.urdf (robot description, URDF)
Before this commit: robot motoman_motomini, 28 links, 27 joints
Links:
- added link leg1, mass 1; collision box size=0.03 0.03 0.7; visual box size=0.03 0.03 0.7
- added link leg2, mass 1; collision box size=0.03 0.03 0.7; visual box size=0.03 0.03 0.7
- added link leg3, mass 1; collision box size=0.03 0.03 0.7; visual box size=0.03 0.03 0.7
- added link leg4, mass 1; collision box size=0.03 0.03 0.7; visual box size=0.03 0.03 0.7
- link table: geometry collision box size=0.83 0.830 0.001; visual box size=0.83 0.830 0.001
Joints:
- added joint leg1_joint: type fixed, parent table, child leg1, origin xyz=0.4 0.4 -0.35 rpy=0.0 0.0 0
- added joint leg2_joint: type fixed, parent table, child leg2, origin xyz=0.4 -0.4 -0.35 rpy=0 0 0
- added joint leg3_joint: type fixed, parent table, child leg3, origin xyz=-0.4 0.4 -0.35 rpy=0 0 0
- added joint leg4_joint: type fixed, parent table, child leg4, origin xyz=-0.4 -0.4 -0.35 rpy=0 0 0
- joint camera_joint: origin xyz=0.903 -0.02 0.52 rpy=0 0.49 -3.14159265359 -> xyz=1.17 0.009 0.52 rpy=0.03 0.49 -3.14159265359
- joint realsense_joint: origin xyz=0.05 0 0.055 rpy=0 -1.57079632679 0 -> xyz=0.05 0 0.055 rpy=0 0 0; parent tool0 -> gripper_base
- joint table_joint: origin xyz=0 -0.1015 0 rpy=0.0 0.0 1.57079632679 -> xyz=0 -0.1015 0.0 rpy=0.0 0.0 1.57079632679

File: motoman/motoman_motomini_support/urdf_old/motomini.xacro (robot description, xacro)
@@ -1,11 +1,10 @@
 <?xml version="1.0" ?>
 <robot name="motoman_motomini" xmlns:xacro="http://ros.org/wiki/xacro">
-  <!--xacro:include filename="$(find motoman_motomini_support)/urdf/motomini_gazebo.xacro" /-->
+  <xacro:include filename="$(find motoman_motomini_support)/urdf/motomini_gazebo.xacro" />
   <xacro:property name="M_PI" value="3.1415926535897931" />
   <xacro:include filename="$(find motoman_motomini_support)/urdf/table_macro.xacro" />
   <xacro:include filename="$(find motoman_motomini_support)/urdf/motomini_macro_kinect1.xacro" />
-  <!--xacro:include filename="$(find motoman_motomini_support)/urdf/gripper_macro.xacro" /-->
+  <xacro:include filename="$(find motoman_motomini_support)/urdf/gripper_macro.xacro" />
   <xacro:include filename="$(find motoman_motomini_support)/urdf/realsense_macro.xacro" />
- <xacro:include filename="$(find robotiq_2f_85_gripper_visualization)/urdf/gripper.xacro"/>
    <!-- World frame -->
   <link name="world" />
@@ -14,14 +13,11 @@
   </xacro:motoman_motomini_table>
   <xacro:motoman_motomini prefix="" parent="table">
-  <origin xyz="0 -0.1015 0" rpy="0.0 0.0 ${M_PI/2}" />
+  <origin xyz="0 -0.1015 0.0" rpy="0.0 0.0 ${M_PI/2}" />
   </xacro:motoman_motomini>
-  <xacro:gripper_mpo prefix="" parent="tool0">
-  <origin xyz="0 0 0" rpy="0 0 -${M_PI/2}" />
-</xacro:gripper_mpo>
-  <!--xacro:motoman_motomini_gripper prefix="" parent="tool0">
+  <xacro:motoman_motomini_gripper prefix="" parent="tool0">
   	<origin xyz="0 0 0" rpy="0 -${M_PI/2} ${M_PI}" />
-  </xacro:motoman_motomini_gripper-->
-  <xacro:motoman_motomini_realsense prefix="" parent="tool0">
-  	<origin xyz="0.05 0 0.055" rpy="0 -${M_PI/2} 0" />
+  </xacro:motoman_motomini_gripper>
+  <xacro:motoman_motomini_realsense prefix="" parent="gripper_base">
+  	<origin xyz="0.05 0 0.055" rpy="0 0 0" />
   </xacro:motoman_motomini_realsense>
 </robot>

File: motoman/motoman_motomini_support/urdf_old/motomini_macro_kinect1.xacro (robot description, xacro)
@@ -171,7 +171,6 @@
     <parent link="${prefix}base_link"/>
     <child link="camera_link"/>
-    <origin xyz="0.903 -0.02 0.52" rpy="0 0.49 ${-M_PI}"/>
+    <origin xyz="1.17 0.009 0.52" rpy="0.03 0.49 ${-M_PI}"/>
 </joint>
-<!--0.91 0.009 0.52 roll 0.03-->
 <joint name="camera_optical_joint" type="fixed">  <!--0.4712 ${{-M_PI/2}-0.4712}-->
     <origin xyz="0 0 0" rpy="${-M_PI/2} 0 ${-M_PI/2}" />
@@ -250,46 +249,58 @@
     <child link="${prefix}base"/>
   </joint>
-<gazebo reference="base_link">
-    <mu1>5.0</mu1>
-    <mu2>5.0</mu2>
-    <material>Gazebo/Blue</material>
-    <turnGravityOff>false</turnGravityOff>
-</gazebo>
-<gazebo reference="${prefix}link_1_s">
-    <mu1>5.0</mu1>
-    <mu2>5.0</mu2>
-    <material>Gazebo/Blue</material>
-    <turnGravityOff>false</turnGravityOff>
-</gazebo>
-<gazebo reference="${prefix}link_2_l">
-    <mu1>5.0</mu1>
-    <mu2>5.0</mu2>
-    <material>Gazebo/Blue</material>
-    <turnGravityOff>false</turnGravityOff>
-</gazebo>
-<gazebo reference="${prefix}link_3_u">
-    <mu1>5.0</mu1>
-    <mu2>5.0</mu2>
-    <material>Gazebo/BlueLaser</material>
-    <turnGravityOff>false</turnGravityOff>
-</gazebo>
-<gazebo reference="${prefix}link_4_r">
-    <mu1>5.0</mu1>
-    <mu2>5.0</mu2>
-    <material>Gazebo/Blue</material>
-    <turnGravityOff>false</turnGravityOff>
-</gazebo>
-<gazebo reference="${prefix}link_5_b">
-    <mu1>5.0</mu1>
-    <mu2>5.0</mu2>
-    <material>Gazebo/Blue</material>
-    <turnGravityOff>false</turnGravityOff>
-</gazebo>
-<gazebo reference="${prefix}link_6_t">
-    <mu1>5.0</mu1>
-    <mu2>5.0</mu2>
-    <material>Gazebo/Blue</material>
-    <turnGravityOff>false</turnGravityOff>
-</gazebo>
+<gazebo reference="joint_1_s">
+    <mu1>5.0</mu1>
+    <mu2>5.0</mu2>
+    <material>Gazebo/Grey</material>
+    <turnGravityOff>false</turnGravityOff>
+</gazebo>
+<gazebo reference="joint_2_l">
+    <mu1>5.0</mu1>
+    <mu2>5.0</mu2>
+    <material>Gazebo/Grey</material>
+    <turnGravityOff>false</turnGravityOff>
+</gazebo>
+<gazebo reference="joint_3_u">
+    <mu1>5.0</mu1>
+    <mu2>5.0</mu2>
+    <material>Gazebo/Grey</material>
+    <turnGravityOff>false</turnGravityOff>
+</gazebo>
+<gazebo reference="joint_4_r">
+    <mu1>5.0</mu1>
+    <mu2>5.0</mu2>
+    <material>Gazebo/Grey</material>
+    <turnGravityOff>false</turnGravityOff>
+</gazebo>
+<gazebo reference="joint_5_b">
+    <mu1>5.0</mu1>
+    <mu2>5.0</mu2>
+    <material>Gazebo/Grey</material>
+    <turnGravityOff>false</turnGravityOff>
+</gazebo>
+<gazebo reference="joint_6_t">
+    <mu1>5.0</mu1>
+    <mu2>5.0</mu2>
+    <material>Gazebo/Grey</material>
+    <turnGravityOff>false</turnGravityOff>
+</gazebo>
+<!--gazebo reference="finger1">
+    <implicitSpringDamper>1</implicitSpringDamper>
+    <kp>1000000.0</kp>
+    <kd>1.0</kd>
+    <mu1>10000.0</mu1>
+    <mu2>10000.0</mu2>
+    <minDepth>0.001</minDepth>
+    <turnGravityOff>false</turnGravityOff>
+</gazebo>
+<gazebo reference="finger2">
+    <implicitSpringDamper>1</implicitSpringDamper>
+    <kp>1000000.0</kp>
+    <kd>1.0</kd>
+    <mu1>100000</mu1>
+    <mu2>100000</mu2>
+    <minDepth>0.001</minDepth>
+    <turnGravityOff>false</turnGravityOff>
+</gazebo-->
 <gazebo reference="camera_link">
     <sensor type="depth" name="camera_1">
@@ -459,9 +470,29 @@
      <hardwareInterface>hardware_interface/PositionJointInterface</hardwareInterface>
     </joint>
-    <actuator name="link6_motor">
+    <actuator name="link5_motor">
      <hardwareInterface>hardware_interface/PositionJointInterface</hardwareInterface>
      <mechanicalReduction>2</mechanicalReduction>
     </actuator>
 </transmission>
+<!--transmission name="link5_finger1_control">
+    <type>transmission_interface/SimpleTransmission</type>
+    <joint name="l_finger_joint">
+     <hardwareInterface>hardware_interface/PositionJointInterface</hardwareInterface>
+    </joint>
+    <actuator name="l_finger_motor">
+     <hardwareInterface>hardware_interface/PositionJointInterface</hardwareInterface>
+     <mechanicalReduction>2</mechanicalReduction>
+    </actuator>
+</transmission>
+<transmission name="link5_finger2_control">
+    <type>transmission_interface/SimpleTransmission</type>
+    <joint name="r_finger_joint">
+     <hardwareInterface>hardware_interface/PositionJointInterface</hardwareInterface>
+    </joint>
+    <actuator name="r_finger_motor">
+     <hardwareInterface>hardware_interface/PositionJointInterface</hardwareInterface>
+     <mechanicalReduction>2</mechanicalReduction>
+    </actuator>
+</transmission-->
   </xacro:macro>
 </robot>

File: motoman/motoman_motomini_support/urdf_old/realsense_macro.xacro (robot description, xacro)
@@ -42,14 +42,4 @@
     <link name="realsense_depth_optical_frame">
   </link>
-<gazebo reference="realsense_link">
-    <implicitSpringDamper>1</implicitSpringDamper>
-    <kp>1000000.0</kp>
-    <kd>1.0</kd>
-    <mu1>10000.0</mu1>
-    <mu2>10000.0</mu2>
-    <minDepth>0.001</minDepth>
-<material>PR2/Grey1</material>
-    <turnGravityOff>true</turnGravityOff>
-</gazebo>
     </xacro:macro>
 </robot>
