Commit message: Relsense Depth fix

File: motoman/motoman_motomini_support/urdf/motoman_motomini.urdf (robot description, URDF)
Before this commit: robot motoman_motomini, 28 links, 27 joints
Joints:
- joint realsense_joint: origin xyz=0.05 0 0.055 rpy=0 -1.57079632679 0 -> xyz=0.05 0 0.055 rpy=0 0 0; parent tool0 -> gripper_base

File: motoman/motoman_motomini_support/urdf/motomini.xacro (robot description, xacro)
@@ -5,7 +5,7 @@
   <xacro:include filename="$(find motoman_motomini_support)/urdf/table_macro.xacro" />
   <xacro:include filename="$(find motoman_motomini_support)/urdf/motomini_macro_kinect1.xacro" />
-  <!--xacro:include filename="$(find motoman_motomini_support)/urdf/gripper_macro.xacro" /-->
+  <xacro:include filename="$(find motoman_motomini_support)/urdf/gripper_macro.xacro" />
   <xacro:include filename="$(find motoman_motomini_support)/urdf/realsense_macro.xacro" />
- <xacro:include filename="$(find robotiq_2f_85_gripper_visualization)/urdf/gripper.xacro"/>
+ <!--xacro:include filename="$(find robotiq_2f_85_gripper_visualization)/urdf/gripper.xacro"/-->
    <!-- World frame -->
   <link name="world" />
@@ -16,12 +16,12 @@
   <origin xyz="0 -0.1015 0" rpy="0.0 0.0 ${M_PI/2}" />
   </xacro:motoman_motomini>
-  <xacro:gripper_mpo prefix="" parent="tool0">
+  <!--xacro:gripper_mpo prefix="" parent="tool0">
   <origin xyz="0 0 0" rpy="0 0 -${M_PI/2}" />
-</xacro:gripper_mpo>
-  <!--xacro:motoman_motomini_gripper prefix="" parent="tool0">
+</xacro:gripper_mpo-->
+  <xacro:motoman_motomini_gripper prefix="" parent="tool0">
   	<origin xyz="0 0 0" rpy="0 -${M_PI/2} ${M_PI}" />
-  </xacro:motoman_motomini_gripper-->
-  <xacro:motoman_motomini_realsense prefix="" parent="tool0">
-  	<origin xyz="0.05 0 0.055" rpy="0 -${M_PI/2} 0" />
+  </xacro:motoman_motomini_gripper>
+  <xacro:motoman_motomini_realsense prefix="" parent="gripper_base">
+  	<origin xyz="0.05 0 0.055" rpy="0 0 0" />
   </xacro:motoman_motomini_realsense>
 </robot>
